Commit message: Update

File: urdf/my_robot.xacro (robot description, xacro)
@@ -2,9 +2,9 @@
   <xacro:include filename="$(find my_robot)/urdf/my_robot.gazebo" />
   <!-- Robot footprint -->
-  <link name="robot_footprint"></link>
+  <link name="robot_footprint"/>
   <joint name="robot_footprint_joint" type="fixed">
-    <origin xyz="0 0 0" rpy="0 0 0" />
+    <origin xyz="0 0 0" rpy="0 0 0"/>
     <parent link="robot_footprint"/>
-    <child link="chassis" />
+    <child link="chassis"/>
   </joint>
   <!-- Chassis link -->
@@ -14,9 +14,5 @@
       <mass value="15.0"/>
       <origin xyz="0.0 0 0" rpy="0 0 0"/>
-      <inertia
-          ixx="0.1" ixy="0" ixz="0"
-          iyy="0.1" iyz="0"
-          izz="0.1"
-      />
+      <inertia ixx="0.1" ixy="0" ixz="0" iyy="0.1" iyz="0" izz="0.1"/>
     </inertial>
     <collision name="collision">
@@ -63,9 +59,5 @@
       <mass value="5"/>
       <origin xyz="0 0 0" rpy="0 1.5707 1.5707"/>
-      <inertia
-          ixx="0.1" ixy="0" ixz="0"
-          iyy="0.1" iyz="0"
-          izz="0.1"
-      />
+      <inertia ixx="0.1" ixy="0" ixz="0" iyy="0.1" iyz="0" izz="0.1"/>
     </inertial>
     <collision name="left_wheel_collision">
@@ -87,9 +79,5 @@
       <mass value="5"/>
       <origin xyz="0 0 0" rpy="0 1.5707 1.5707"/>
-      <inertia
-          ixx="0.1" ixy="0" ixz="0"
-          iyy="0.1" iyz="0"
-          izz="0.1"
-      />
+      <inertia ixx="0.1" ixy="0" ixz="0" iyy="0.1" iyz="0" izz="0.1"/>
     </inertial>
     <collision name="right_wheel_collision">
@@ -126,15 +114,9 @@
   <!-- Camera Link -->
   <link name="camera">
-    <!-- Inertial Properties -->
     <inertial>
       <mass value="0.1"/>
       <origin xyz="0.05 0.05 0.05" rpy="0 0 0"/>
-      <inertia
-          ixx="1e-6" ixy="0" ixz="0"
-          iyy="1e-6" iyz="0"
-          izz="1e-6"
-      />
-    </inertial>
-    <!-- Collision Properties -->
+      <inertia ixx="1e-6" ixy="0" ixz="0" iyy="1e-6" iyz="0" izz="1e-6"/>
+    </inertial>
     <collision>
       <origin xyz="0 0 0" rpy="0 0 0"/>
@@ -143,5 +125,4 @@
       </geometry>
     </collision>
-    <!-- Visual Properties -->
     <visual>
       <origin xyz="0 0 0" rpy="0 0 0"/>
@@ -160,15 +141,9 @@
   <!-- Hokuyo Lidar Link -->
   <link name="hokuyo">
-    <!-- Inertial Properties -->
     <inertial>
       <mass value="1e-5"/>
       <origin xyz="0 0 0" rpy="0 0 0"/>
-      <inertia
-          ixx="1e-6" ixy="0" ixz="0"
-          iyy="1e-6" iyz="0"
-          izz="1e-6"
-      />
-    </inertial>
-    <!-- Collision Properties -->
+      <inertia ixx="1e-6" ixy="0" ixz="0" iyy="1e-6" iyz="0" izz="1e-6"/>
+    </inertial>
     <collision>
       <origin xyz="0 0 0" rpy="0 0 0"/>
@@ -177,9 +152,7 @@
       </geometry>
     </collision>
-    <!-- Visual Properties -->
     <visual>
       <origin xyz="0 0 0" rpy="0 0 0"/>
       <geometry>
-        <!-- Path to the mesh file -->
         <mesh filename="package://my_robot/meshes/hokuyo.dae"/>
       </geometry>
@@ -193,4 +166,32 @@
     <axis xyz="0 1 0"/>
   </joint>
+  <!-- Differential Drive Plugin -->
+  <gazebo>
+    <plugin name="differential_drive_controller" filename="libgazebo_ros_diff_drive.so">
+      <legacyMode>false</legacyMode>
+      <alwaysOn>true</alwaysOn>
+      <updateRate>10</updateRate>
+      <leftJoint>left_wheel_hinge</leftJoint>
+      <rightJoint>right_wheel_hinge</rightJoint>
+      <wheelSeparation>0.3</wheelSeparation>
+      <wheelDiameter>0.2</wheelDiameter>
+      <torque>10</torque>
+      <commandTopic>cmd_vel</commandTopic>
+      <odometryTopic>odom</odometryTopic>
+      <odometryFrame>odom</odometryFrame>
+      <robotBaseFrame>robot_footprint</robotBaseFrame>
+      <publishWheelTF>true</publishWheelTF>
+      <publishWheelJointState>true</publishWheelJointState>
+      <publishTf>1</publishTf>
+      <publishOdomTF>true</publishOdomTF>
+      <odometrySource>world</odometrySource>
+    </plugin>
+    <!-- Hokuyo Laser Plugin -->
+    <plugin name="gazebo_ros_head_hokuyo_controller" filename="libgazebo_ros_laser.so">
+      <topicName>/my_robot/laser/scan</topicName>
+      <frameName>hokuyo</frameName>
+    </plugin>
+  </gazebo>
+  <!-- Materials -->
   <gazebo reference="left_wheel">
     <material>Gazebo/Green</material>
